File: Simple E-ink Display .kicad_pcb (KiCad board)
At the start: 2 copper layers, 59.2 x 29 mm, 16 parts, among them J1 Conn_01x10_Male, J2 Conn_01x24_Female, J3 Conn_01x10_Male

Commit message: rev 2.1
Parts:
- added H1: MountingHole, MountingHole:MountingHole_2.1mm, F.Cu at (123.9, 109.1)
- added H2: MountingHole, MountingHole:MountingHole_2.1mm, F.Cu at (168.5, 86.0)
- added H3: MountingHole, MountingHole:MountingHole_2.1mm, F.Cu at (124.0, 86.2)
- added H4: MountingHole, MountingHole:MountingHole_2.1mm, F.Cu at (168.4, 109.0)
- added J4: Conn_01x06_Female, AeonLabs:pogo 6pin magnetic, F.Cu at (154.6, 97.7)
- J1: value Conn_01x10_Male -> Conn_01x06_Female; footprint Connector_PinSocket_2.54mm:PinSocket_1x10_P2.54mm_Horizontal -> AeonLabs:pogo 6pin magnetic
- moved G*** 29.3 mm to (133.1, 109.3)
- moved G*** 28.1 mm to (135.9, 96.3)
- moved FPC5 22.3 mm to (148.1, 90.3), turned to 90 degrees
- moved FPC4 18.5 mm to (145.7, 90.3), turned to 90 degrees
- moved J1 12.8 mm to (116.3, 97.6), turned to 90 degrees
- moved G*** 4.23 mm to (132.3, 103.0)
- moved FPC18 3.21 mm to (131.6, 90.5)
- moved FPC19 3.19 mm to (134.1, 90.5)
- moved FPC16 3.19 mm to (127.0, 90.4)
- moved FPC17 3.19 mm to (129.3, 90.5)
- moved FPC20 3.19 mm to (136.4, 90.5)
- moved FPC22 3.19 mm to (138.8, 90.4)
- moved FPC23 3.19 mm to (141.1, 90.4)
- moved FPC24 3.19 mm to (143.3, 90.3)
- moved J2 0.69 mm to (161.4, 97.6)
Routing:
- net /GND: track 143.7 -> 89.3 mm
- net /3V3: track 62.7 -> 33.1 mm
- net /RESE: track 58.4 -> 30.2 mm
- net /GDR: track 42.2 -> 19.8 mm
- net Net-(FPC16-Pad1): track 31.5 -> 51.8 mm, vias 0 -> 2
- net Net-(FPC17-Pad1): track 28.5 -> 46.3 mm, vias 0 -> 2
- net /SDI: track 83.6 -> 99.5 mm, vias 0 -> 2
- net Net-(FPC18-Pad1): track 25.9 -> 41.8 mm, vias 0 -> 2
- net /PREVGL: track 93.7 -> 107.7 mm, vias 0 -> 2
- net /PREVGH: track 91.0 -> 79.2 mm, vias 1 -> 4
- net Net-(FPC19-Pad1): track 23.3 -> 34.5 mm, vias 0 -> 2
- net Net-(FPC20-Pad1): track 20.9 -> 31.8 mm, vias 0 -> 2
- net Net-(FPC22-Pad1): track 18.5 -> 28.8 mm, vias 0 -> 2
- net /RES: track 73.2 -> 64.7 mm, vias 0 -> 2
- net /VCOM: track 13.2 -> 20.7 mm, vias 0 -> 2
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Other:
- board text added: "59x29mm rev. 2.0"
- board text added: "DATA PINS"
- board text added: "POWER PINS"
- board text added: "To Upload an Image to the E-ink Display connect to AeonLabs E-Ink Configuration Device (E-Ink CD)"
- board text removed: "59x29mm rev. 1.0"
- board text removed: "To Configure an Image on the E-ink Display connect J1/J3 to AeonLabs E-Ink Configuration Device (E-Ink CD)"
- board text removed: "www.aeoonlabs.solutions"
