File: Simple E-ink Display .kicad_sch (KiCad schematic)
At the start: 13 parts, among them J1 Conn_01x10_Male, J2 Conn_01x24_Female, J3 Conn_01x10_Male

Commit message: rev 2.1
Parts:
- removed J1: Conn_01x10_Male, Connector_PinSocket_2.54mm:PinSocket_1x10_P2.54mm_Horizontal, symbol Connector:Conn_01x10_Male
- added H1, H2, H3, H4: MountingHole, MountingHole:MountingHole_2.1mm, symbol Mechanical:MountingHole
- added J1, J4: Conn_01x06_Female, AeonLabs:pogo 6pin magnetic, symbol Connector:Conn_01x06_Female
Connections:
- net 3V3: now also J4.2 (Pin_2)
- net CS: now also J1.5 (Pin_5)
- net GDR: now also J4.4 (Pin_4)
- net GND: now also J4.1 (Pin_1)
- net PREVGH: now also J1.2 (Pin_2)
- net PREVGL: now also J1.1 (Pin_1)
- net RES: now also J1.6 (Pin_6)
- net RESE: now also J4.3 (Pin_3)
- net SCLK: now also J1.4 (Pin_4)
- net SDI: now also J1.3 (Pin_3)
- no-connect marks 4 -> 6
Other:
- moved on the sheet: J3
